File: ProductionPCB/pcbs/pnpL.kicad_pcb (KiCad board)
At the start: 2 copper layers, 167 x 122.9 mm, 63 parts

Commit message: rev 1.1
Connections:
- T1 pad 1: Bplus -> (no net)
- T1 pad 2: (no net) -> Bplus
Routing:
- net Bplus: track 39.5 -> 38.3 mm
Other:
- board text added: "NICE!NANO FACE DOWN"
Changed lines of the file:
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@@
     (pad "" smd rect (at 3.7 -1.1 270) (size 0.9 0.9) (layers "F.Cu" "F.Paste" "F.Mask"))
     (pad "" smd rect (at 3.7 1.1 270) (size 0.9 0.9) (layers "F.Cu" "F.Paste" "F.Mask"))
-    (pad "1" smd rect (at 2.25 2.075 270) (size 0.9 1.25) (layers "F.Cu" "F.Paste" "F.Mask")
+    (pad "1" smd rect (at 2.25 2.075 270) (size 0.9 1.25) (layers "F.Cu" "F.Paste" "F.Mask"))
+    (pad "2" smd rect (at -0.75 2.075 270) (size 0.9 1.25) (layers "F.Cu" "F.Paste" "F.Mask")
       (net 52 "Bplus"))
-    (pad "2" smd rect (at -0.75 2.075 270) (size 0.9 1.25) (layers "F.Cu" "F.Paste" "F.Mask"))
     (pad "3" smd rect (at -2.25 2.075 270) (size 0.9 1.25) (layers "F.Cu" "F.Paste" "F.Mask")
       (net 41 "RAW"))
@@
   (gr_arc (start 168.66474 137.048556) (mid 164.894911 139.663456) (end 160.347345 139.056032)
     (stroke (width 0.15) (type solid)) (layer "Edge.Cuts"))
+  (gr_text "NICE!NANO FACE DOWN\n" (at 145.796 42.418 90) (layer "F.SilkS")
+    (effects (font (size 1 1) (thickness 0.15)) (justify left bottom))
+  )
   (segment (start 26.49 92.91) (end 25.4133 92.91) (width 0.25) (layer "F.Cu") (net 1))
   (segment (start 25.4133 92.91) (end 25.4133 91.8332) (width 0.25) (layer "F.Cu") (net 1))
@@
   (segment (start 157.565 83.66) (end 155.6037 83.66) (width 0.25) (layer "F.Cu") (net 41))
   (segment (start 155.6037 83.66) (end 155.2286 83.2849) (width 0.25) (layer "F.Cu") (net 41))
-  (segment (start 157.1037 85.16) (end 157.565 85.16) (width 0.25) (layer "F.Cu") (net 41))
   (via (at 155.2286 83.2849) (size 0.8) (drill 0.4) (layers "F.Cu" "B.Cu") (net 41))
   (segment (start 140.6108 50.9013) (end 138.3366 53.1755) (width 0.25) (layer "B.Cu") (net 41))
@@
   (segment (start 142.36 54.81) (end 142.36 53.3333) (width 0.25) (layer "B.Cu") (net 49))
   (segment (start 142.1457 53.119) (end 142.1457 42.2143) (width 0.25) (layer "B.Cu") (net 49))
-  (segment (start 136.6633 58.91) (end 136.6633 66.3025) (width 0.25) (layer "F.Cu") (net 52))
-  (segment (start 157.4441 87.0833) (end 157.565 87.0833) (width 0.25) (layer "F.Cu") (net 52))
-  (segment (start 138.14 58.91) (end 136.6633 58.91) (width 0.25) (layer "F.Cu") (net 52))
-  (segment (start 136.6633 66.3025) (end 157.4441 87.0833) (width 0.25) (layer "F.Cu") (net 52))
-  (segment (start 157.565 88.16) (end 157.565 87.0833) (width 0.25) (layer "F.Cu") (net 52))
+  (segment (start 136.6633 58.91) (end 138.14 58.91) (width 0.25) (layer "F.Cu") (net 52))
+  (segment (start 154.248 85.16) (end 136.6633 67.5753) (width 0.25) (layer "F.Cu") (net 52))
+  (segment (start 136.6633 67.5753) (end 136.6633 58.91) (width 0.25) (layer "F.Cu") (net 52))
+  (segment (start 157.565 85.16) (end 154.248 85.16) (width 0.25) (layer "F.Cu") (net 52))
   (group "" (id 2a57a11a-0fb2-432a-9d30-ebe07179c1ff)
     (members
